File: octotemp/hardware/OctoTemp.kicad_pcb (KiCad board)
At the start: 2 copper layers, 47.2 x 34 mm, 42 parts, among them P1 CONN_02X03, P2 CONN_01X02, P3 CONN_01X08, P4 CONN_01X08, U1 ESP-12E, U2 SPX3819M5, U3 ADC128D818

Commit message: Added name/version silkscreening.
Other:
- board text added: "z2amiller OctoTemp v0.3.1"
Changed lines of the file:
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@@
     (area 15.514536 18.70288 75.926201 56.65218)
     (thickness 1.6)
-    (drawings 5)
+    (drawings 6)
     (tracks 269)
     (zones 0)
@@
     )
   )
+  (gr_text "z2amiller OctoTemp v0.3.1" (at 66.55 36.128 90) (layer B.SilkS)
+    (effects (font (size 1.5 1.5) (thickness 0.3)) (justify mirror))
+  )
   (gr_circle (center 22.55 31.528) (end 22.55 31.928) (layer F.SilkS) (width 0.2))
